File: stupid-mobility-adapter-v3/stupid-mobility-adapter-v3/stupid-mobility-adapter-v3.kicad_sch (KiCad schematic)
At the start: 38 parts, among them J1 BTS7968-0, J10 UART, J2 Act0-FB, J3 BTS7968-1, J4 Act1-FB, J5 ESTOP_INPUT, J6 UART, J7 Relays, J8 I2C, J9 BATT_MON_SELECT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

Commit message: build and setup board for v4.1/4.1
Parts:
- J9: footprint Connector_PinSocket_2.54mm:PinSocket_1x03_P2.54mm_Vertical -> Connector_PinHeader_2.54mm:PinHeader_1x03_P2.54mm_Vertical
Connections:
- net Buzz: now reaches R14.2
- net Buzz: now also U5.14 (GPIO35)
- no-connect marks 15 -> 14
Changed lines of the file:
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@@
   (no_connect (at 50.8 34.29))
   (no_connect (at 201.93 147.32))
-  (no_connect (at 199.39 121.92))
   (no_connect (at 102.87 35.56))
   (no_connect (at 90.17 35.56))
@@
     (effects (font (size 1.27 1.27)) (justify left bottom))
   )
+  (label "Buzz" (at 199.39 121.92 180)
+    (effects (font (size 1.27 1.27)) (justify right bottom))
+  )
   (label "ESTOP_IN" (at 199.39 114.3 180)
     (effects (font (size 1.27 1.27)) (justify right bottom))
@@
   (label "TX" (at 246.38 119.38 0)
     (effects (font (size 1.27 1.27)) (justify left bottom))
+  )
+  (label "Buzz" (at 262.89 139.7 180)
+    (effects (font (size 1.27 1.27)) (justify right bottom))
   )
   (label "ACT0_FB" (at 35.56 62.23 180)
@@
       (effects (font (size 1.27 1.27)) (justify left))
     )
-    (property "Footprint" "Connector_PinSocket_2.54mm:PinSocket_1x03_P2.54mm_Vertical" (id 2) (at 198.12 83.82 0)
+    (property "Footprint" "Connector_PinHeader_2.54mm:PinHeader_1x03_P2.54mm_Vertical" (id 2) (at 198.12 83.82 0)
       (effects (font (size 1.27 1.27)) hide)
     )
@@
     )
     (path "/c3e3b447-1acd-4f6c-a522-0cc6e96c7d76"
-      (reference "J9") (unit 1) (value "BATT_MON_SELECT") (footprint "Connector_PinSocket_2.54mm:PinSocket_1x03_P2.54mm_Vertical")
+      (reference "J9") (unit 1) (value "BATT_MON_SELECT") (footprint "Connector_PinHeader_2.54mm:PinHeader_1x03_P2.54mm_Vertical")
     )
     (path "/c06ee988-6065-4d85-b30f-f7b82e32170d"
